File: AES72-4E.kicad_pcb (KiCad board)
At the start: 2 copper layers, 50 x 38 mm, 5 parts, among them J101 NSJ12HC, J102 NSJ12HC, J103 NE8FAH

Commit message: Replace Order_Number
Parts:
- INFO101: value Order_Number -> ~; footprint V2_Production:Order_Number -> V2_Production:Revision
Changed lines of the file:
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@@
-			)
-		)
-		(property "Mouser" "568-NE8FAH"
-			(at 0 0 90)
-			(unlocked yes)
-			(layer "F.Fab")
-			(hide yes)
-			(effects
-				(font
-					(size 1 1)
-					(thickness 0.15)
-				)
-			)
-		)
-		(property "Manufacturer" "Neutrik"
-			(at 0 0 90)
-			(unlocked yes)
-			(layer "F.Fab")
-			(hide yes)
-			(effects
-				(font
-					(size 1 1)
-					(thickness 0.15)
-				)
-			)
-		)
-		(property "Product" "NE8FAH"
-			(at 0 0 90)
-			(unlocked yes)
-			(layer "F.Fab")
-			(hide yes)
-			(effects
-				(font
-					(size 1 1)
-					(thickness 0.15)
-				)
 			)
 		)
@@
 			)
 		)
-		(property "Datasheet" "https://www.neutrik.com/en/product/nsj12hc"
+		(property "Datasheet" ""
 			(at -20.48 -8.5 0)
 			(unlocked yes)
@@
 			)
 		)
-		(property "Description" "Stacking Jacks, Stereo dual jack, full nose"
+		(property "Description" ""
 			(at -20.48 -8.5 0)
 			(unlocked yes)
@@
 				(font
 					(size 1.27 1.27)
-					(thickness 0.15)
-				)
-			)
-		)
-		(property "Mouser" "568-NSJ12HC"
-			(at 0 0 0)
-			(unlocked yes)
-			(layer "F.Fab")
-			(hide yes)
-			(effects
-				(font
-					(size 1 1)
-					(thickness 0.15)
-				)
-			)
-		)
-		(property "Manufacturer" "Neutrik"
-			(at 0 0 0)
-			(unlocked yes)
-			(layer "F.Fab")
-			(hide yes)
-			(effects
-				(font
-					(size 1 1)
-					(thickness 0.15)
-				)
-			)
-		)
-		(property "Product" "NSJ12HC"
-			(at 0 0 0)
-			(unlocked yes)
-			(layer "F.Fab")
-			(hide yes)
-			(effects
-				(font
-					(size 1 1)
 					(thickness 0.15)
 				)
@@
 		)
 		(embedded_fonts no)
-		(model "../../../versioduo.kicad/3dmodels/V2_Connector_Audio.3dshapes/NSJ12HC.step"
+		(model "../../3dmodels/V2_Connector_Audio.3dshapes/NSJ12HC.step"
 			(offset
 				(xyz -0.28 0 23)
@@
 			)
 		)
-		(property "Datasheet" "https://www.neutrik.com/en/product/nsj12hc"
+		(property "Datasheet" ""
 			(at -20.48 -8.5 0)
 			(unlocked yes)
@@
 			)
 		)
-		(property "Description" "Stacking Jacks, Stereo dual jack, full nose"
+		(property "Description" ""
 			(at -20.48 -8.5 0)
 			(unlocked yes)
@@
 				(font
 					(size 1.27 1.27)
-					(thickness 0.15)
-				)
-			)
-		)
-		(property "Mouser" "568-NSJ12HC"
-			(at 0 0 0)
-			(unlocked yes)
-			(layer "F.Fab")
-			(hide yes)
-			(effects
-				(font
-					(size 1 1)
-					(thickness 0.15)
-				)
-			)
-		)
-		(property "Manufacturer" "Neutrik"
-			(at 0 0 0)
-			(unlocked yes)
-			(layer "F.Fab")
-			(hide yes)
-			(effects
-				(font
-					(size 1 1)
-					(thickness 0.15)
-				)
-			)
-		)
-		(property "Product" "NSJ12HC"
-			(at 0 0 0)
-			(unlocked yes)
-			(layer "F.Fab")
-			(hide yes)
-			(effects
-				(font
-					(size 1 1)
 					(thickness 0.15)
 				)
@@
 		)
 		(embedded_fonts no)
-		(model "../../../versioduo.kicad/3dmodels/V2_Connector_Audio.3dshapes/NSJ12HC.step"
+		(model "../../3dmodels/V2_Connector_Audio.3dshapes/NSJ12HC.step"
 			(offset
 				(xyz -0.28 0 23)
@@
 		(embedded_fonts no)
 	)
-	(footprint "V2_Production:Order_Number"
+	(footprint "V2_Production:Revision"
 		(layer "B.Cu")
 		(at 64.5 98.707107 90)
@@
 			)
 		)
-		(property "Value" "Order_Number"
+		(property "Value" "~"
 			(at 0 -2.27 270)
 			(unlocked yes)
@@
 		(sheetname "/")
 		(sheetfile "AES72-4E.kicad_sch")
-		(attr exclude_from_pos_files exclude_from_bom)
-		(fp_rect
-			(start -7 0.75)
-			(end 7 -0.75)
-			(stroke
-				(width 0.05)
-				(type default)
-			)
-			(fill no)
-			(layer "B.CrtYd")
-		)
-		(fp_text user "${Order-Number}"
+		(attr exclude_from_pos_files exclude_from_bom allow_missing_courtyard)
+		(fp_text user "${REVISION} (${ISSUE_DATE})"
 			(at 0 0 270)
 			(unlocked yes)
@@
 			(effects
 				(font
-					(size 0.8 0.8)
-					(thickness 0.12)
+					(size 0.75 0.75)
+					(thickness 0.1)
 				)
 				(justify mirror)
+			)
+		)
+		(fp_text user "${REVISION} (${ISSUE_DATE})"
+			(at 0 0 270)
+			(unlocked yes)
+			(layer "B.Fab")
+			(effects
+				(font
+					(size 0.75 0.75)
+					(thickness 0.1)
+				)
+				(justify mirror)
