File: AES72-4E.kicad_sch (KiCad schematic)
At the start: 5 parts, among them J101 NSJ12HC, J102 NSJ12HC, J103 NE8FAH

Commit message: Update
Parts:
- INFO101: value ~ -> (none)
- J101, J102: Id (none) -> Audio:${SYMBOL_NAME}; Rating (none) -> 6.35mm
- J103: Id (none) -> EtherCon:${SYMBOL_NAME}; Rating (none) -> CAT5e
